File: ergogen/output/pcbs/clackr-right.kicad_pcb (KiCad board)
At the start: 2 copper layers, 140.7 x 125.3 mm, 99 parts

Commit message: reset right side
Parts:
- removed the REF** at (259.2, -6.21)
- removed the REF** at (278.3, -68.1)
- removed the REF** at (199.3, -46.2)
- removed the REF** at (238.8, -5.76)
- removed the REF** at (278.3, -87.2)
- removed the REF** at (316.3, -17.4)
- removed the REF** at (218.8, -1.77)
- removed the REF** at (240.3, -49.1)
- removed the REF** at (221.3, -46.2)
- removed the REF** at (278.3, -30.0)
- removed the REF** at (316.3, 1.60)
- removed the REF** at (278.3, -49.1)
- removed the REF** at (259.3, -53.8)
- removed the REF** at (297.3, -74.6)
- removed the REF** at (221.3, -84.3)
- removed the REF** at (259.3, -34.8)
- removed the REF** at (240.3, -68.1)
- removed the REF** at (221.3, -65.3)
- removed the REF** at (316.3, -74.6)
- removed the REF** at (316.3, -36.5)
- removed the REF** at (297.3, -17.4)
- removed the REF** at (221.3, -27.2)
- removed the REF** at (297.3, -55.5)
- removed the REF** at (316.3, -55.5)
- removed the REF** at (259.3, -91.9)
- removed the REF** at (240.3, -87.2)
- removed the REF** at (240.3, -30.0)
- removed the REF** at (259.3, -72.9)
- removed the REF** at (297.3, -36.5)
- removed the REF** at (297.3, 1.60)
- removed the REF** at (199.8, 5.64)
- added REF**: VIA-0.6mm, VIA-0.6mm, F.Cu at (316.3, 1.60)
- added REF**: VIA-0.6mm, VIA-0.6mm, F.Cu at (297.3, -74.6)
- added REF**: VIA-0.6mm, VIA-0.6mm, F.Cu at (278.3, -30.0)
- added REF**: VIA-0.6mm, VIA-0.6mm, F.Cu at (278.3, -49.1)
- added REF**: VIA-0.6mm, VIA-0.6mm, F.Cu at (278.3, -68.1)
- added REF**: VIA-0.6mm, VIA-0.6mm, F.Cu at (278.3, -87.2)
- added REF**: VIA-0.6mm, VIA-0.6mm, F.Cu at (259.3, -34.8)
- added REF**: VIA-0.6mm, VIA-0.6mm, F.Cu at (259.3, -53.8)
- added REF**: VIA-0.6mm, VIA-0.6mm, F.Cu at (259.3, -72.9)
- added REF**: VIA-0.6mm, VIA-0.6mm, F.Cu at (259.3, -91.9)
- added REF**: VIA-0.6mm, VIA-0.6mm, F.Cu at (240.3, -30.0)
- added REF**: VIA-0.6mm, VIA-0.6mm, F.Cu at (316.3, -17.4)
- added REF**: VIA-0.6mm, VIA-0.6mm, F.Cu at (240.3, -49.1)
- added REF**: VIA-0.6mm, VIA-0.6mm, F.Cu at (240.3, -68.1)
- added REF**: VIA-0.6mm, VIA-0.6mm, F.Cu at (240.3, -87.2)
- added REF**: VIA-0.6mm, VIA-0.6mm, F.Cu at (221.3, -27.2)
- added REF**: VIA-0.6mm, VIA-0.6mm, F.Cu at (221.3, -46.2)
- added REF**: VIA-0.6mm, VIA-0.6mm, F.Cu at (221.3, -65.3)
- added REF**: VIA-0.6mm, VIA-0.6mm, F.Cu at (221.3, -84.3)
- added REF**: VIA-0.6mm, VIA-0.6mm, F.Cu at (259.2, -6.21)
- added REF**: VIA-0.6mm, VIA-0.6mm, F.Cu at (238.8, -5.76)
- added REF**: VIA-0.6mm, VIA-0.6mm, F.Cu at (218.8, -1.77)
- added REF**: VIA-0.6mm, VIA-0.6mm, F.Cu at (316.3, -36.5)
- added REF**: VIA-0.6mm, VIA-0.6mm, F.Cu at (199.8, 5.64)
- added REF**: VIA-0.6mm, VIA-0.6mm, F.Cu at (199.3, -46.2)
- added REF**: VIA-0.6mm, VIA-0.6mm, F.Cu at (316.3, -55.6)
- added REF**: VIA-0.6mm, VIA-0.6mm, F.Cu at (316.3, -74.6)
- added REF**: VIA-0.6mm, VIA-0.6mm, F.Cu at (297.3, 1.60)
- added REF**: VIA-0.6mm, VIA-0.6mm, F.Cu at (297.3, -17.4)
- added REF**: VIA-0.6mm, VIA-0.6mm, F.Cu at (297.3, -36.5)
- added REF**: VIA-0.6mm, VIA-0.6mm, F.Cu at (297.3, -55.6)
Routing:
- net P1: track 379.3 -> 0.00 mm
- net P0: track 375.6 -> 0.00 mm
- net P2: track 310.3 -> 0.00 mm
- net P3: track 293.0 -> 0.00 mm
- net P5: track 233.3 -> 0.00 mm
- net P15: track 218.1 -> 0.00 mm
- net P14: track 187.4 -> 0.00 mm
- net P4: track 183.1 -> 0.00 mm
- net P18: track 166.8 -> 0.00 mm
- net P16: track 160.1 -> 0.00 mm, vias 2 -> 0
- net P19: track 151.0 -> 0.00 mm
- net P20: track 141.9 -> 0.00 mm
- net GND: track 106.2 -> 0.00 mm
- net RE_A: track 34.5 -> 0.00 mm
- net RST: track 33.1 -> 0.00 mm
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