File: ergogen/output/pcbs/clackr-left-completed.kicad_pcb (KiCad board)
At the start: 2 copper layers, 140.7 x 125.3 mm, 99 parts

Commit message: update all outlines
Parts:
- removed the REF** at (232.3, 188.7)
- removed the REF** at (134.9, 173.0)
- removed the REF** at (191.9, 98.5)
- removed the REF** at (153.9, 134.9)
- removed the REF** at (229.9, 144.2)
- removed the REF** at (210.9, 122.3)
- removed the REF** at (191.9, 184.3)
- removed the REF** at (191.9, 155.7)
- removed the REF** at (229.9, 106.2)
- removed the REF** at (172.9, 141.4)
- removed the REF** at (134.9, 154.0)
- removed the REF** at (172.9, 160.4)
- removed the REF** at (229.9, 125.2)
- removed the REF** at (212.3, 184.7)
- removed the REF** at (153.9, 154.0)
- removed the REF** at (191.9, 117.6)
- removed the REF** at (191.9, 136.6)
- removed the REF** at (210.9, 141.4)
- removed the REF** at (210.9, 103.3)
- removed the REF** at (134.9, 134.9)
- removed the REF** at (251.9, 144.2)
- removed the REF** at (153.9, 173.0)
- removed the REF** at (134.9, 192.1)
- removed the REF** at (153.9, 115.9)
- removed the REF** at (134.9, 115.9)
- removed the REF** at (251.3, 196.1)
- removed the REF** at (172.9, 122.3)
- removed the REF** at (229.9, 163.3)
- removed the REF** at (210.9, 160.4)
- removed the REF** at (153.9, 192.1)
- removed the REF** at (172.9, 103.3)
- added MH1: , ceoloide:mounting_hole_npth, F.Cu at (9.47, -9.53)
- added MH2: , ceoloide:mounting_hole_npth, F.Cu at (9.47, -66.7)
- added MH3: , ceoloide:mounting_hole_npth, F.Cu at (47.5, -45.9)
- added MH4: , ceoloide:mounting_hole_npth, F.Cu at (47.5, -84.0)
- added MH5: , ceoloide:mounting_hole_npth, F.Cu at (85.5, -38.3)
- added MH6: , ceoloide:mounting_hole_npth, F.Cu at (85.5, -76.4)
- added MH7: , ceoloide:mounting_hole_npth, F.Cu at (117.0, -19.2)
- added REF**: VIA-0.6mm, VIA-0.6mm, F.Cu at (30.4, -49.1)
- added REF**: VIA-0.6mm, VIA-0.6mm, F.Cu at (89.9, -1.77)
- added REF**: VIA-0.6mm, VIA-0.6mm, F.Cu at (11.4, 1.60)
- added REF**: VIA-0.6mm, VIA-0.6mm, F.Cu at (11.4, -55.5)
- added REF**: VIA-0.6mm, VIA-0.6mm, F.Cu at (49.4, -91.9)
- added REF**: VIA-0.6mm, VIA-0.6mm, F.Cu at (11.4, -74.6)
- added REF**: VIA-0.6mm, VIA-0.6mm, F.Cu at (49.4, -53.8)
- added REF**: VIA-0.6mm, VIA-0.6mm, F.Cu at (-7.60, -74.6)
- added REF**: VIA-0.6mm, VIA-0.6mm, F.Cu at (68.4, -49.1)
- added REF**: VIA-0.6mm, VIA-0.6mm, F.Cu at (69.8, -5.76)
- added REF**: VIA-0.6mm, VIA-0.6mm, F.Cu at (30.4, -30.0)
- added REF**: VIA-0.6mm, VIA-0.6mm, F.Cu at (30.4, -87.2)
- added REF**: VIA-0.6mm, VIA-0.6mm, F.Cu at (108.9, 5.64)
- added REF**: VIA-0.6mm, VIA-0.6mm, F.Cu at (87.4, -65.3)
- added REF**: VIA-0.6mm, VIA-0.6mm, F.Cu at (87.4, -84.3)
- added REF**: VIA-0.6mm, VIA-0.6mm, F.Cu at (87.4, -27.2)
- added REF**: VIA-0.6mm, VIA-0.6mm, F.Cu at (-7.60, 1.60)
- added REF**: VIA-0.6mm, VIA-0.6mm, F.Cu at (11.4, -36.5)
- added REF**: VIA-0.6mm, VIA-0.6mm, F.Cu at (-7.60, -36.5)
- added REF**: VIA-0.6mm, VIA-0.6mm, F.Cu at (49.5, -6.21)
- added REF**: VIA-0.6mm, VIA-0.6mm, F.Cu at (109.4, -46.2)
- added REF**: VIA-0.6mm, VIA-0.6mm, F.Cu at (68.4, -68.1)
- added REF**: VIA-0.6mm, VIA-0.6mm, F.Cu at (-7.60, -17.4)
- added REF**: VIA-0.6mm, VIA-0.6mm, F.Cu at (11.4, -17.4)
- added REF**: VIA-0.6mm, VIA-0.6mm, F.Cu at (87.4, -46.2)
- added REF**: VIA-0.6mm, VIA-0.6mm, F.Cu at (-7.60, -55.5)
- added REF**: VIA-0.6mm, VIA-0.6mm, F.Cu at (30.4, -68.1)
- added REF**: VIA-0.6mm, VIA-0.6mm, F.Cu at (49.4, -34.8)
- added REF**: VIA-0.6mm, VIA-0.6mm, F.Cu at (49.4, -72.9)
- added REF**: VIA-0.6mm, VIA-0.6mm, F.Cu at (68.4, -30.0)
- added REF**: VIA-0.6mm, VIA-0.6mm, F.Cu at (68.4, -87.2)
- moved D12 237.8 mm to (45.6, -49.1)
- moved D13 237.8 mm to (45.6, -68.1)
- moved D14 237.8 mm to (45.6, -87.2)
- moved D15 237.8 mm to (64.6, -34.8)
- moved D18 237.8 mm to (64.6, -91.9)
- moved D20 237.8 mm to (83.6, -49.1)
- moved D21 237.8 mm to (83.6, -68.1)
- moved D22 237.8 mm to (83.6, -87.2)
- moved D23 237.8 mm to (102.6, -27.2)
- moved D25 237.8 mm to (102.6, -65.3)
- moved D26 237.8 mm to (102.6, -84.3)
- moved D29 237.8 mm to (104.1, 3.43)
- moved D4 237.8 mm to (7.60, -55.5)
- moved D9 237.8 mm to (26.6, -55.5)
- moved RE1 237.8 mm to (117.0, -47.8)
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Routing:
- net P14: track 253.5 -> 168.8 mm
- net P5: track 211.8 -> 177.0 mm
- net P15: track 273.3 -> 240.9 mm
- net P19: track 191.3 -> 161.3 mm
- net P18: track 212.3 -> 187.9 mm
- net P2: track 295.2 -> 277.6 mm
- net P0: track 349.1 -> 332.2 mm
- net P3: track 278.7 -> 264.1 mm
- net P1: track 361.1 -> 349.3 mm
- net RAW: track 28.6 -> 18.0 mm
- net P20: track 170.4 -> 165.4 mm
- net GND: track 90.2 -> 94.7 mm, vias 0 -> 1
- net MOSI: track 16.6 -> 12.1 mm
- net P4: track 164.1 -> 159.9 mm
- net SCK: track 10.6 -> 14.0 mm
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Other:
- outline, holes or cut-outs redrawn
- board text added: "clackr"
- board text removed: "CS"
