File: ergogen/output/pcbs/clackr-right-completed.kicad_pcb (KiCad board)
At the start: 2 copper layers, 140.7 x 125.3 mm, 99 parts

Commit message: update all outlines
Parts:
- added MH1: , ceoloide:mounting_hole_npth, F.Cu at (299.2, -9.53)
- added MH2: , ceoloide:mounting_hole_npth, F.Cu at (299.2, -66.7)
- added MH3: , ceoloide:mounting_hole_npth, F.Cu at (261.2, -45.9)
- added MH4: , ceoloide:mounting_hole_npth, F.Cu at (261.2, -84.0)
- added MH5: , ceoloide:mounting_hole_npth, F.Cu at (223.2, -38.3)
- added MH6: , ceoloide:mounting_hole_npth, F.Cu at (223.2, -76.4)
- added MH7: , ceoloide:mounting_hole_npth, F.Cu at (191.7, -19.2)
Routing:
- net P5: track 233.3 -> 194.9 mm
- net RAW: track 25.5 -> 63.0 mm
- net GND: track 106.2 -> 81.2 mm, vias 0 -> 1
- net RST: track 33.1 -> 50.4 mm
- net P4: track 183.1 -> 176.1 mm
- net MOSI: track 18.6 -> 12.1 mm
- net P1: track 379.3 -> 373.5 mm
- net BAT_P: track 15.5 -> 21.0 mm, vias 0 -> 1
- net P0: track 375.6 -> 370.4 mm
- net P2: track 310.3 -> 314.7 mm
- net SCK: track 10.6 -> 14.0 mm
- net P20: track 141.9 -> 139.4 mm
- net P19: track 151.0 -> 148.8 mm
- net P18: track 166.8 -> 164.8 mm
- net RE_C: track 26.1 -> 24.5 mm
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Other:
- outline, holes or cut-outs redrawn
- board text added: "by hackr"
